File: macropad_kicad/macropad_kicad.kicad_pcb (KiCad board)
At the start: 2 copper layers, 81 x 90.5 mm, 28 parts, among them J1 OLED_128x64, SW1 RotaryEncoder_Switch, U1 MOUDLE-SEEEDUINO-XIAO

Commit message: added that copper cool effect thing
Routing:
- added copper zone on B.Cu, net (none)
- added copper zone on F.Cu, net (none)
Changed lines of the file:
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@@
 		(net 25)
+	)
+	(zone
+		(net 0)
+		(net_name "")
+		(layers "F&B.Cu")
+		(hatch edge 0.5)
+		(connect_pads
+			(clearance 0.5)
+		)
+		(min_thickness 0.25)
+		(filled_areas_thickness no)
+		(fill yes
+			(thermal_gap 0.5)
+			(thermal_bridge_width 0.5)
+			(island_removal_mode 1)
+			(island_area_min 10)
+		)
+		(polygon
+			(pts
+				(xy 140.49375 16.66875) (xy 140.49375 116.68125) (xy 47.625 116.68125) (xy 47.625 16.66875)
+			)
+		)
 	)
 	(generated
